Commit message: Added Joint, Caster Wheel Link, Caste wheel Support, caster wheel of both left and right wheel, Tires, hubcab part.

File: src/robot_description/urdf/robot.urdf (robot description, URDF)
Before this commit: robot robot, 1 links, 0 joints
Links:
- added link link_caster_wheel, mass 1; collision sphere radius=0.10; collision sphere radius=0.2
- added link link_left_wheel, mass 1; collision cylinder length=0.12 radius=0.08; collision cylinder length=0.12 radius=0.4
- added link link_right_wheel, mass 1; collision cylinder length=0.12 radius=0.08; collision cylinder length=0.12 radius=0.4
Joints:
- added joint joint_chassis_caster_wheel: type fixed, parent link_chassis, child link_caster_wheel, origin xyz=0.8 0 -0.15 rpy=0 0 0
- added joint joint_chassis_left_wheel: type continuous, parent link_chassis, child link_left_wheel, origin xyz=-0.5 0.65 0 rpy=0 0 0, axis 0 1 0, limit effort=10000 velocity=1000
- added joint joint_chassis_right_wheel: type continuous, parent link_chassis, child link_right_wheel, origin xyz=-0.5 -0.65 0 rpy=0 0 0, axis 0 1 0, limit effort=10000 velocity=1000
