Commit message: Added tail parts

File: src/robot_description/urdf/robot.xacro (robot description, xacro)
@@ -226,3 +226,44 @@
         </collision>
     </link>
+      <!-- Robot tail -->
+      <joint name="joint_tail" type="continuous">
+        <origin rpy="0 0 0" xyz="-1 0 0" />
+        <child link="link_tail" />
+        <axis rpy="0 0 0" xyz="0 1 0" />
+        <parent link="link_chassis" />
+        <joint_properties damping="1.0" friction="1.0" />
+    </joint>
+    <link name="link_tail">
+        <inertial>
+            <origin xyz="0 0 0" rpy="0 0 0" />
+            <mass value="0.5" />
+            <inertia ixx="0.000252666666667" ixy="0" ixz="0" iyy="0.000252666666667" iyz="0" izz="0.0005"/>
+        </inertial>
+        <visual>
+            <origin xyz="-0.2 0 0" rpy="0 ${pi/2} 0" />
+            <geometry>
+                <cylinder radius="0.05" length="0.40"/>
+            </geometry>
+            <material name="Red">
+                <color rgba="0.7 0.1 0.1 1" />
+            </material>
+        </visual>
+        <collision>
+            <origin xyz="-0.2 0 0" rpy="0 ${pi/2} 0"/>
+            <geometry>
+                <cylinder radius="0.05" length="0.40"/>
+            </geometry>
+        </collision>
+    </link>
+    <!-- Transmission -->
+    <transmission name="tran_tail">
+        <type>transmission_interface/SimpleTransmission</type>
+        <joint name="joint_tail">
+            <hardwareInterface>hardware_interface/EffortJointInterface</hardwareInterface>
+        </joint>
+        <actuator name="motor_joint_tail">
+            <hardwareInterface>hardware_interface/EffortJointInterface</hardwareInterface>
+            <mechanicalReduction>1</mechanicalReduction>
+        </actuator>
+    </transmission>
 </robot>

Commit message: Changed xacro file for camera module

File: src/robot_description/urdf/robot.xacro (robot description, xacro)
@@ -1,269 +1,311 @@
-<?xml version="1.0" ?>
+<?xml version="1.0"?>
 <robot name="robot" xmlns:xacro="http://www.ros.org/wiki/xacro">
-    <xacro:include filename="$(find robot_description)/urdf/robot.gazebo" />
-    <!-- Parameters -->
-    <xacro:property name="chassis_mass" value="10" />
-    <xacro:property name="pi" value="3.1415926535897931"/>
-    <!-- Link - chassis -->
-    <link name="link_chassis">
-        <inertial>
-            <mass value="${chassis_mass}" />
-            <origin xyz="0 0 0.3" rpy="0 0 0" />
-            <inertia ixx="1.5417" ixy="0" ixz="0" iyy="3.467" iyz="0" izz="4.742" />
-        </inertial>
-        <collision>
-            <!-- <geometry>
-                <box size="2 1.3 0.4" />
-            </geometry> -->
-            <geometry>
-                <mesh filename="package://robot_description/meshes/chassis.stl" />
-            </geometry>
-        </collision>
-        <visual>
-            <geometry>
-                <mesh filename="package://robot_description/meshes/chassis.stl" />
-            </geometry>
-            <!-- <geometry>
-                <box size="2 1.3 0.4" />
-            </geometry> -->
-            <material name="DarkBlue">
-                <color rgba="0.2 0.2 0.4 1" />
-            </material>
-        </visual>
-    </link>
-    <!-- Joint - caster wheel -->
-    <joint name="joint_chassis_caster_wheel" type="fixed">
-        <origin rpy="0 0 0" xyz="0.8 0 -0.15" />
-        <child link="link_caster_wheel" />
-        <parent link="link_chassis" />
-        <joint_properties damping="1.0" friction="1.0" />
-    </joint>
-    <!-- Link - caster wheel -->
-    <link name="link_caster_wheel">
-        <inertial>
-            <mass value="1" />
-            <origin xyz="0 0 0" rpy="0 0 0" />
-            <inertia ixx="0.002526666666667" ixy="0" ixz="0" iyy="0.002526666666667" iyz="0" izz="0.005"/>
-        </inertial>
-        <!-- Caster wheel support -->
-        <collision>
-            <origin rpy="0 0 0" xyz="0 0 -0.03" />
-            <geometry>
-                <sphere radius="0.2" />
-            </geometry>
-        </collision>
-        <visual>
-            <origin rpy="0 0 0" xyz="0 0 -0.03" />
-            <geometry>
-                <sphere radius="0.2" />
-            </geometry>
-            <material name="DarkBlue">
-                <color rgba="0.2 0.2 0.4 1" />
-            </material>
-        </visual>
-        <!-- Caster wheel -->
-        <collision>
-            <origin rpy="0 0 0" xyz="0 0 -0.15" />
-            <geometry>
-                <sphere radius="0.10" />
-            </geometry>
-        </collision>
-        <visual>
-            <origin rpy="0 0 0" xyz="0 0 -0.15" />
-            <geometry>
-                <sphere radius="0.10" />
-            </geometry>
-            <material name="Grey">
-                <color rgba="0.6 0.6 0.6 1" />
-            </material>
-        </visual>
-    </link>
-    <!-- Joint - chassis / left wheel -->
-    <joint name="joint_chassis_left_wheel" type="continuous">
-        <origin rpy="0 0 0" xyz="-0.5 0.65 0" />
-        <child link="link_left_wheel" />
-        <parent link="link_chassis" />
-        <axis rpy="0 0 0" xyz="0 1 0" />
-        <limit effort="10000" velocity="1000" />
-        <joint_properties damping="1.0" friction="1.0" />
-    </joint>
-    <!-- Link - left wheel -->
-    <link name="link_left_wheel">
-        <inertial>
-            <mass value="1" />
-            <origin xyz="0 0 0" rpy="0 0 0" />
-            <inertia ixx="0.002526666666667" ixy="0" ixz="0" iyy="0.002526666666667" iyz="0" izz="0.005"/>
-        </inertial>
-        <!-- Tires -->
-        <collision>
-            <origin rpy="${pi/2} 0 0" xyz="0 0.18 0" />
-            <geometry>
-                <cylinder length="0.12" radius="0.4"/>
-            </geometry>
-        </collision>
-        <visual>
-            <origin rpy="${pi/2} 0 0" xyz="0 0.18 0" />
-            <geometry>
-                <mesh filename="package://robot_description/meshes/wheel.stl" />
-            </geometry>
-            <material name="Black">
-                <color rgba="0.1 0.1 0.1 1" />
-            </material>
-        </visual>
-        <!-- Axle -->
-        <collision>
-            <origin rpy="${pi/2} 0 0" xyz="0 0.06 0" />
-            <geometry>
-                <cylinder length="0.12" radius="0.08"/>
-            </geometry>
-        </collision>
-        <visual>
-            <origin rpy="${pi/2} 0 0" xyz="0 0.06 0" />
-            <geometry>
-                <cylinder length="0.12" radius="0.08"/>
-            </geometry>
-            <material name="Grey">
-                <color rgba="0.6 0.6 0.6 1" />
-            </material>
-        </visual>
-        <!-- Hubcap -->
-        <visual>
-            <origin rpy="${pi/2} 0 0" xyz="0 0.18 0" />
-            <geometry>
-                <box size="0.02 0.5 0.02" />
-            </geometry>
-            <material name="Grey">
-                <color rgba="0.6 0.6 0.6 1" />
-            </material>
-        </visual>
-    </link>
-    <!-- Joint - chassis / right wheel -->
-    <joint name="joint_chassis_right_wheel" type="continuous">
-        <origin rpy="0 0 0" xyz="-0.5 -0.65 0" />
-        <child link="link_right_wheel" />
-        <parent link="link_chassis" />
-        <axis rpy="0 0 0" xyz="0 1 0" />
-        <limit effort="10000" velocity="1000" />
-        <joint_properties damping="1.0" friction="1.0" />
-    </joint>
-    <!-- Link - right wheel -->
-    <link name="link_right_wheel">
-        <inertial>
-            <mass value="1" />
-            <origin xyz="0 0 0" rpy="0 0 0" />
-            <inertia ixx="0.002526666666667" ixy="0" ixz="0" iyy="0.002526666666667" iyz="0" izz="0.005"/>
-        </inertial>
-        <!-- Tires -->
-        <collision>
-            <origin rpy="${pi/2} 0 0" xyz="0 -0.18 0" />
-            <geometry>
-                <cylinder length="0.12" radius="0.4"/>
-            </geometry>
-        </collision>
-        <visual>
-            <origin rpy="${pi/2} 0 0" xyz="0 -0.18 0" />
-            <geometry>
-                <mesh filename="package://robot_description/meshes/wheel.stl" />
-            </geometry>
-            <material name="Black">
-                <color rgba="0.1 0.1 0.1 1" />
-            </material>
-        </visual>
-        <!-- Axle -->
-        <collision>
-            <origin rpy="${pi/2} 0 0" xyz="0 -0.06 0" />
-            <geometry>
-                <cylinder length="0.12" radius="0.08"/>
-            </geometry>
-        </collision>
-        <visual>
-            <origin rpy="${pi/2} 0 0" xyz="0 -0.06 0" />
-            <geometry>
-                <cylinder length="0.12" radius="0.08"/>
-            </geometry>
-            <material name="Grey">
-                <color rgba="0.6 0.6 0.6 1" />
-            </material>
-        </visual>
-        <!-- Hubcap -->
-        <visual>
-            <origin rpy="${pi/2} 0 0" xyz="0 -0.18 0" />
-            <geometry>
-                <box size="0.02 0.5 0.02" />
-            </geometry>
-            <material name="Grey">
-                <color rgba="0.6 0.6 0.6 1" />
-            </material>
-        </visual>
-    </link>
-    <!-- Laser scan -->
-    <joint name="joint_laser_scan_chassis" type="fixed">
-        <origin rpy="0 0 0" xyz="0.8 0 0.3" />
-        <child link="link_laser_scan" />
-        <parent link="link_chassis" />
-        <joint_properties damping="1.0" friction="1.0" />
-    </joint>
-    <link name="link_laser_scan">
-        <inertial>
-            <origin xyz="0 0 0" rpy="0 0 0" />
-            <mass value="0.5" />
-            <inertia ixx="0.000252666666667" ixy="0" ixz="0" iyy="0.000252666666667" iyz="0" izz="0.0005"/>
-        </inertial>
-        <visual>
-            <origin xyz="0 0 0" rpy="0 0 0" />
-            <geometry>
-                <cylinder radius="0.15" length="0.20"/>
-            </geometry>
-            <material name="Red">
-                <color rgba="0.7 0.1 0.1 1" />
-            </material>
-        </visual>
-        <collision>
-            <origin xyz="0 0 0" rpy="0 0 0"/>
-            <geometry>
-                <cylinder radius="0.15" length="0.20"/>
-            </geometry>
-        </collision>
-    </link>
-      <!-- Robot tail -->
-      <joint name="joint_tail" type="continuous">
-        <origin rpy="0 0 0" xyz="-1 0 0" />
-        <child link="link_tail" />
-        <axis rpy="0 0 0" xyz="0 1 0" />
-        <parent link="link_chassis" />
-        <joint_properties damping="1.0" friction="1.0" />
-    </joint>
-    <link name="link_tail">
-        <inertial>
-            <origin xyz="0 0 0" rpy="0 0 0" />
-            <mass value="0.5" />
-            <inertia ixx="0.000252666666667" ixy="0" ixz="0" iyy="0.000252666666667" iyz="0" izz="0.0005"/>
-        </inertial>
-        <visual>
-            <origin xyz="-0.2 0 0" rpy="0 ${pi/2} 0" />
-            <geometry>
-                <cylinder radius="0.05" length="0.40"/>
-            </geometry>
-            <material name="Red">
-                <color rgba="0.7 0.1 0.1 1" />
-            </material>
-        </visual>
-        <collision>
-            <origin xyz="-0.2 0 0" rpy="0 ${pi/2} 0"/>
-            <geometry>
-                <cylinder radius="0.05" length="0.40"/>
-            </geometry>
-        </collision>
-    </link>
-    <!-- Transmission -->
-    <transmission name="tran_tail">
-        <type>transmission_interface/SimpleTransmission</type>
-        <joint name="joint_tail">
-            <hardwareInterface>hardware_interface/EffortJointInterface</hardwareInterface>
-        </joint>
-        <actuator name="motor_joint_tail">
-            <hardwareInterface>hardware_interface/EffortJointInterface</hardwareInterface>
-            <mechanicalReduction>1</mechanicalReduction>
-        </actuator>
-    </transmission>
+	<include filename="$(find robot_description)/urdf/robot.gazebo" />
+	<!-- Parameters -->
+	<property name="pi" value="3.1415926535897931" />
+	<xacro:property name="camera_link" value="1.05" />
+	<xacro:property name="chassis_mass" value="10" />
+	<xacro:property name="camera_size" value="0.1" />
+	<!-- Link - chassis -->
+	<link name="link_chassis">
+		<inertial>
+			<mass value="${chassis_mass}" />
+			<origin xyz="0 0 0.3" rpy="0 0 0" />
+			<inertia ixx="1.5417" ixy="0" ixz="0" iyy="3.467" iyz="0" izz="4.742" />
+		</inertial>
+		<collision>
+			<!--
+			<geometry>
+			<box size="2 1.3 0.4" />
+			</geometry>
+			-->
+			<geometry>
+				<mesh filename="package://robot_description/meshes/chassis.stl" />
+			</geometry>
+		</collision>
+		<visual>
+			<geometry>
+				<mesh filename="package://robot_description/meshes/chassis.stl" />
+			</geometry>
+			<!--
+			<geometry>
+			<box size="2 1.3 0.4" />
+			</geometry>
+			-->
+			<material name="DarkBlue">
+				<color rgba="0.2 0.2 0.4 1" />
+			</material>
+		</visual>
+	</link>
+	<!-- Joint - caster wheel -->
+	<joint name="joint_chassis_caster_wheel" type="fixed">
+		<origin rpy="0 0 0" xyz="0.8 0 -0.15" />
+		<child link="link_caster_wheel" />
+		<parent link="link_chassis" />
+		<joint_properties damping="1.0" friction="1.0" />
+	</joint>
+	<!-- Link - caster wheel -->
+	<link name="link_caster_wheel">
+		<inertial>
+			<mass value="1" />
+			<origin xyz="0 0 0" rpy="0 0 0" />
+			<inertia ixx="0.002526666666667" ixy="0" ixz="0" iyy="0.002526666666667" iyz="0" izz="0.005" />
+		</inertial>
+		<!-- Caster wheel support -->
+		<collision>
+			<origin rpy="0 0 0" xyz="0 0 -0.03" />
+			<geometry>
+				<sphere radius="0.2" />
+			</geometry>
+		</collision>
+		<visual>
+			<origin rpy="0 0 0" xyz="0 0 -0.03" />
+			<geometry>
+				<sphere radius="0.2" />
+			</geometry>
+			<material name="DarkBlue">
+				<color rgba="0.2 0.2 0.4 1" />
+			</material>
+		</visual>
+		<!-- Caster wheel -->
+		<collision>
+			<origin rpy="0 0 0" xyz="0 0 -0.15" />
+			<geometry>
+				<sphere radius="0.10" />
+			</geometry>
+		</collision>
+		<visual>
+			<origin rpy="0 0 0" xyz="0 0 -0.15" />
+			<geometry>
+				<sphere radius="0.10" />
+			</geometry>
+			<material name="Grey">
+				<color rgba="0.6 0.6 0.6 1" />
+			</material>
+		</visual>
+	</link>
+	<!-- Joint - chassis / left wheel -->
+	<joint name="joint_chassis_left_wheel" type="continuous">
+		<origin rpy="0 0 0" xyz="-0.5 0.65 0" />
+		<child link="link_left_wheel" />
+		<parent link="link_chassis" />
+		<axis rpy="0 0 0" xyz="0 1 0" />
+		<limit effort="10000" velocity="1000" />
+		<joint_properties damping="1.0" friction="1.0" />
+	</joint>
+	<!-- Link - left wheel -->
+	<link name="link_left_wheel">
+		<inertial>
+			<mass value="1" />
+			<origin xyz="0 0 0" rpy="0 0 0" />
+			<inertia ixx="0.002526666666667" ixy="0" ixz="0" iyy="0.002526666666667" iyz="0" izz="0.005" />
+		</inertial>
+		<!-- Tires -->
+		<collision>
+			<origin rpy="${pi/2} 0 0" xyz="0 0.18 0" />
+			<geometry>
+				<cylinder length="0.12" radius="0.4" />
+			</geometry>
+		</collision>
+		<visual>
+			<origin rpy="${pi/2} 0 0" xyz="0 0.18 0" />
+			<geometry>
+				<mesh filename="package://robot_description/meshes/wheel.stl" />
+			</geometry>
+			<material name="Black">
+				<color rgba="0.1 0.1 0.1 1" />
+			</material>
+		</visual>
+		<!-- Axle -->
+		<collision>
+			<origin rpy="${pi/2} 0 0" xyz="0 0.06 0" />
+			<geometry>
+				<cylinder length="0.12" radius="0.08" />
+			</geometry>
+		</collision>
+		<visual>
+			<origin rpy="${pi/2} 0 0" xyz="0 0.06 0" />
+			<geometry>
+				<cylinder length="0.12" radius="0.08" />
+			</geometry>
+			<material name="Grey">
+				<color rgba="0.6 0.6 0.6 1" />
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